File: hardware/ece_souvenir.kicad_sch (KiCad schematic)
At the start: 37 parts, among them U1 TLC555CDR

Commit message: feat(sch): pick C1 basic X5R part, add keychain hole H1, add logo art
C1 -> C52923 (1uF 25V X5R 0402, JLC basic) instead of extended X7R to
avoid a loading fee; temp range irrelevant for a souvenir. H1 2.5 mm
NPTH keychain hole added so board and schematic stay in parity.
art/ece_logo.png is the source raster for the top silkscreen.

Co-Authored-By: Claude Opus 5.5 <noreply@anthropic.com>
Parts:
- added H1: Keychain, MountingHole:MountingHole_2.5mm, symbol Mechanical:MountingHole
- C1: footprint Capacitor_SMD:C_0603_1608Metric -> Capacitor_SMD:C_0402_1005Metric; LCSC C106248 -> C52923; MPN CC0603KRX7R7BB105 -> CL05A105KA5NQNC
Changed lines of the file:
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@@
 			)
 		)
-		(property "Footprint" "Capacitor_SMD:C_0603_1608Metric"
+		(property "Footprint" "Capacitor_SMD:C_0402_1005Metric"
 			(at 71.12 76.2 0)
 			(hide yes)
@@
 			)
 		)
-		(property "Description" "1 uF 16 V X7R 0603, timing"
+		(property "Description" "1 uF 25 V X5R 0402, timing"
 			(at 71.12 76.2 0)
 			(hide yes)
@@
 			)
 		)
-		(property "LCSC" "C106248"
+		(property "LCSC" "C52923"
 			(at 71.12 76.2 0)
 			(hide yes)
@@
 			)
 		)
-		(property "MPN" "CC0603KRX7R7BB105"
+		(property "MPN" "CL05A105KA5NQNC"
 			(at 71.12 76.2 0)
 			(hide yes)
@@
 					(unit 1)
 				)
+			)
+		)
+	)
+	(symbol
+		(lib_id "Mechanical:MountingHole")
+		(at 193.04 96.52 0)
+		(unit 1)
+		(body_style 1)
+		(exclude_from_sim no)
+		(in_bom yes)
+		(on_board yes)
+		(in_pos_files yes)
+		(dnp no)
+		(property "Reference" "H1"
+			(at 195.58 95.25 0)
+			(show_name no)
+			(do_not_autoplace no)
+			(effects
+				(font
+					(size 1.27 1.27)
+				)
+				(justify left)
+			)
+		)
+		(property "Value" "Keychain"
+			(at 195.58 97.79 0)
+			(show_name no)
+			(do_not_autoplace no)
+			(effects
+				(font
+					(size 1.27 1.27)
+				)
+				(justify left)
+			)
+		)
+		(property "Footprint" "MountingHole:MountingHole_2.5mm"
+			(at 193.04 96.52 0)
+			(hide yes)
+			(show_name no)
+			(do_not_autoplace no)
+			(effects
+				(font
+					(size 1.27 1.27)
+				)
+			)
+		)
+		(property "Datasheet" ""
+			(at 193.04 96.52 0)
+			(hide yes)
+			(show_name no)
+			(do_not_autoplace no)
+			(effects
+				(font
+					(size 1.27 1.27)
+				)
+			)
+		)
+		(property "Description" "2.5 mm NPTH keychain hole"
+			(at 193.04 96.52 0)
+			(hide yes)
+			(show_name no)
+			(do_not_autoplace no)
+			(effects
+				(font
+					(size 1.27 1.27)
+				)
+			)
+		)
+		(property "LCSC" ""
+			(at 193.04 96.52 0)
+			(hide yes)
+			(show_name no)
+			(do_not_autoplace no)
+			(effects
+				(font
+					(size 1.27 1.27)
+				)
+			)
+		)
+		(property "MPN" ""
+			(at 193.04 96.52 0)
+			(hide yes)
+			(show_name no)
+			(do_not_autoplace no)
+			(effects
+				(font
+					(size 1.27 1.27)
+				)
+			)
+		)
+		(instances
+			(project "ece_souvenir"
+				(path "/6c3e6f0e-5b1a-4c55-9e0e-ece500000001"
+					(reference "H1")
+					(unit 1)
+				)

Commit message: feat(pcb): board outline, keychain hole, logo silk and bottom placement
30x30 mm R1 outline, 2.5 mm NPTH at (27,3). Logo traced from
art/ece_logo.png into 48 F.SilkS polygons (24 x 21.3 mm). All parts on
bottom: LEDs per spec 7-segment table (x mirrored), series resistors
parallel to each LED, U1 at 270 deg with C2 1.96 mm from pin 8.
JLCPCB rules and Power net class written to .kicad_pro.

DRC: 0 violations, 0 parity issues, 57 unconnected (routing pending).

Co-Authored-By: Claude Opus 5.5 <noreply@anthropic.com>
Parts:
- H1, TP1, TP2, TP3: now left out of the parts list
Changed lines of the file:
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@@
 		(body_style 1)
 		(exclude_from_sim no)
-		(in_bom yes)
+		(in_bom no)
 		(on_board yes)
 		(in_pos_files yes)
@@
 			)
 		)
-		(property "LCSC" ""
-			(at 193.04 73.66 0)
-			(hide yes)
-			(show_name no)
-			(do_not_autoplace no)
-			(effects
-				(font
-					(size 1.27 1.27)
-				)
-			)
-		)
-		(property "MPN" ""
-			(at 193.04 73.66 0)
-			(hide yes)
-			(show_name no)
-			(do_not_autoplace no)
-			(effects
-				(font
-					(size 1.27 1.27)
-				)
-			)
-		)
 		(pin "1"
 		)
@@
 		(body_style 1)
 		(exclude_from_sim no)
-		(in_bom yes)
+		(in_bom no)
 		(on_board yes)
 		(in_pos_files yes)
@@
 			)
 		)
-		(property "LCSC" ""
-			(at 180.34 73.66 0)
-			(hide yes)
-			(show_name no)
-			(do_not_autoplace no)
-			(effects
-				(font
-					(size 1.27 1.27)
-				)
-			)
-		)
-		(property "MPN" ""
-			(at 180.34 73.66 0)
-			(hide yes)
-			(show_name no)
-			(do_not_autoplace no)
-			(effects
-				(font
-					(size 1.27 1.27)
-				)
-			)
-		)
 		(pin "1"
 		)
@@
 		(body_style 1)
 		(exclude_from_sim no)
-		(in_bom yes)
+		(in_bom no)
 		(on_board yes)
 		(in_pos_files yes)
@@
 			)
 		)
-		(property "LCSC" ""
-			(at 167.64 73.66 0)
-			(hide yes)
-			(show_name no)
-			(do_not_autoplace no)
-			(effects
-				(font
-					(size 1.27 1.27)
-				)
-			)
-		)
-		(property "MPN" ""
-			(at 167.64 73.66 0)
-			(hide yes)
-			(show_name no)
-			(do_not_autoplace no)
-			(effects
-				(font
-					(size 1.27 1.27)
-				)
-			)
-		)
 		(pin "1"
 		)
@@
 		(body_style 1)
 		(exclude_from_sim no)
-		(in_bom yes)
+		(in_bom no)
 		(on_board yes)
 		(in_pos_files yes)
@@
 			(at 193.04 96.52 0)
 			(hide yes)
-			(show_name no)
-			(do_not_autoplace no)
-			(effects
-				(font
-					(size 1.27 1.27)
-				)
-			)
-		)
-		(property "LCSC" ""
-			(at 193.04 96.52 0)
-			(hide yes)
-			(show_name no)
-			(do_not_autoplace no)
-			(effects
-				(font
-					(size 1.27 1.27)
-				)
-			)
-		)
-		(property "MPN" ""
-			(at 193.04 96.52 0)
-			(hide yes)

Commit message: feat(pcb): switch to 0603 hand-solder parts and re-place
All parts will be hand soldered, so nothing smaller than 0603: LEDs
XL-1608UOC-06 (C965800), passives 0603 with KiCad HandSolder footprints.
C1 back to X7R (Yageo C106248) per the original spec now that JLC
basic/extended fees no longer apply. Series resistors moved inside each
digit to fit the larger 0603 courtyards.

ERC 0, netlist OK. DRC: 0 violations, 0 parity, 57 unconnected (routing
pending).

Co-Authored-By: Claude Opus 5.5 <noreply@anthropic.com>
Parts:
- C1: footprint Capacitor_SMD:C_0402_1005Metric -> Capacitor_SMD:C_0603_1608Metric_Pad1.08x0.95mm_HandSolder; LCSC C52923 -> C106248; MPN CL05A105KA5NQNC -> CC0603KRX7R7BB105
- C2: footprint Capacitor_SMD:C_0402_1005Metric -> Capacitor_SMD:C_0603_1608Metric_Pad1.08x0.95mm_HandSolder; LCSC C1525 -> C14663; MPN CL05B104KO5NNNC -> CC0603KRX7R9BB104
- C3: footprint Capacitor_SMD:C_0402_1005Metric -> Capacitor_SMD:C_0603_1608Metric_Pad1.08x0.95mm_HandSolder; LCSC C15195 -> C57112; MPN CL05B103KB5NNNC -> 0603B103K500NT
- D1, D10, D11, D12, D13, D14, D2, D3, D4, D5, D6, D7, D8, D9: footprint LED_SMD:LED_0402_1005Metric -> LED_SMD:LED_0603_1608Metric_Pad1.05x0.95mm_HandSolder; LCSC C965791 -> C965800; MPN XL-1005UOC -> XL-1608UOC-06
- R1: footprint Resistor_SMD:R_0402_1005Metric -> Resistor_SMD:R_0603_1608Metric_Pad0.98x0.95mm_HandSolder; LCSC C26083 -> C22935; MPN 0402WGF1004TCE -> 0603WAF1004T5E
- R10, R11, R12, R13, R14, R15, R16, R3, R4, R5, R6, R7, R8, R9: footprint Resistor_SMD:R_0402_1005Metric -> Resistor_SMD:R_0603_1608Metric_Pad0.98x0.95mm_HandSolder; LCSC C25890 -> C22978; MPN 0402WGF3301TCE -> 0603WAF3301T5E
- R2: footprint Resistor_SMD:R_0402_1005Metric -> Resistor_SMD:R_0603_1608Metric_Pad0.98x0.95mm_HandSolder; LCSC C25750 -> C25808; MPN 0402WGF1203TCE -> 0603WAF1203T5E

Commit message: feat(sch): PNP high-side LED driver, one resistor per digit
Advisor review 2026-10-11:
- Q1 MMBT3906LT1G (C53444) PNP high-side switch, base via R6 4.7k from
  555 OUT. On while OUT is LOW, so the 9.7 % flash duty is kept; the 555
  now supplies ~0.55-0.9 mA base current instead of sinking ~13 mA.
- One current-limit resistor per digit: R3/R5 680R (E, 5 LEDs), R4 820R
  (C, 4 LEDs) = 3.3k/n, same average per-LED current. 14 -> 3 resistors.
- LED cathodes now to GND; new nets OUT, LED_PWR, A_E1, A_C, A_E2.

ERC 0 errors / 0 warnings; netlist matches spec (tools/check_netlist.py).

Co-Authored-By: Claude Opus 5.5 <noreply@anthropic.com>
Parts:
- removed R10, R11, R12, R13, R14, R15, R16, R7, R8, R9: 3.3k, Resistor_SMD:R_0603_1608Metric_Pad0.98x0.95mm_HandSolder, symbol Device:R
- added Q1: MMBT3906, Package_TO_SOT_SMD:SOT-23_Handsoldering, symbol Transistor_BJT:Q_PNP_BEC
- R3, R5: value 3.3k -> 680; LCSC C22978 -> C23228; MPN 0603WAF3301T5E -> 0603WAF6800T5E
- R4: value 3.3k -> 820; LCSC C22978 -> C23253; MPN 0603WAF3301T5E -> 0603WAF8200T5E
- R6: value 3.3k -> 4.7k; LCSC C22978 -> C23162; MPN 0603WAF3301T5E -> 0603WAF4701T5E
Connections:
- net GND: now also D1.1 (K), D10.1 (K), D11.1 (K), D12.1 (K), D13.1 (K), D14.1 (K), D2.1 (K), D3.1 (K), D4.1 (K), D5.1 (K), D6.1 (K), D7.1 (K), D8.1 (K), D9.1 (K)
- net VCC: now also Q1.2 (E); no longer R3.1, R4.1, R5.1, R6.1
- net A_E2: now reaches D10.2 (A)
- net A_E2: now also D11.2 (A), D12.2 (A), D13.2 (A), D14.2 (A), R5.2
- net A_E1: now reaches D1.2 (A), R3.2
- net A_E1: now also D2.2 (A), D3.2 (A), D4.2 (A), D5.2 (A)
- net A_C: now reaches D9.2 (A)
- net A_C: now also D6.2 (A), D7.2 (A), D8.2 (A), R4.2
- net OUT: now reaches R6.2
- net OUT: now also TP3.1, U1.3 (OUT); no longer D4.2 (A)
- removed net LED_SINK: D1.1 (K), D10.1 (K), D11.1 (K), D12.1 (K), D13.1 (K), D14.1 (K), D2.1 (K), D3.1 (K), D4.1 (K), D5.1 (K), D6.1 (K), D7.1 (K), D8.1 (K), D9.1 (K), TP3.1, U1.3 (OUT)
- new net: Q1.1 (B), R6.1
- new net LED_PWR: Q1.3 (C), R3.1, R4.1, R5.1
Other:
- note added: "Astable 555. Q1 (PNP) turns on while OUT is LOW (discharge phase). t_on = 0.693 * R2 * C1 = 83 ms t_off = 0.693 * (R1 + R2) * C1 = 776 ms f = 1.16 Hz, LED duty 9.7 % I_digit = (VCC - Vce_sat - Vf) / R: E 680R, C 820R -> ~0.4 mA @3.3 V ... ~0.9 mA @5 V average per LED (shared, unballasted) Q1 base: (VCC - Veb) / 4.7k = 0.55 ... 0.9 mA, forced beta >= 10"
- note removed: "Astable 555, LEDs lit while OUT is LOW (discharge phase). t_on = 0.693 * R2 * C1 = 83 ms t_off = 0.693 * (R1 + R2) * C1 = 776 ms f = 1.16 Hz, LED duty 9.7 % I_LED = (VCC - Vf - V_OL) / 3.3k = 0.4 mA @3.3 V ... 0.9 mA @5 V each"
- moved on the sheet: D1, D10, D11, D12, D13, D14, D2, D3, D4, D5, D6, D7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

Commit message: feat: white LEDs for letter C, R4 220R, R6 3.3k
D6-D9 -> XINGLIGHT XL-1608UWC-04 white (C965808). White Vf ~2.6 V at
~1 mA leaves ~0.65 V headroom at 3.3 V, so R4 drops 820R -> 220R
(C22962) to keep C brightness close to the orange E's from 3.3 V to 5 V
(~5-17 mcd vs ~6-14 mcd). Q1 load rises to ~19.5 mA at 5 V, so R6
4.7k -> 3.3k (C22978) for forced beta ~9-15.

Re-routed (same pipeline): 297.8 mm B.Cu, 0 F.Cu, 0 vias. DRC rule
min_resolved_spokes 1 (pour is supplementary; all pads have traces).
ERC 0/0, netlist OK, DRC 0/0/0, EMI audit PASS.

Co-Authored-By: Claude Opus 5.5 <noreply@anthropic.com>
Parts:
- D6, D7, D8, D9: value Orange -> White; LCSC C965800 -> C965808; MPN XL-1608UOC-06 -> XL-1608UWC-04
- R4: value 820 -> 220; LCSC C23253 -> C22962; MPN 0603WAF8200T5E -> 0603WAF2200T5E
- R6: value 4.7k -> 3.3k; LCSC C23162 -> C22978; MPN 0603WAF4701T5E -> 0603WAF3301T5E
Other:
- note added: "Astable 555. Q1 (PNP) turns on while OUT is LOW (discharge phase). t_on = 0.693 * R2 * C1 = 83 ms t_off = 0.693 * (R1 + R2) * C1 = 776 ms f = 1.16 Hz, LED duty 9.7 % I_digit = (VCC - Vce_sat - Vf) / R: E (orange) 680R, C (white) 220R orange ~0.4 mA @3.3 V ... ~0.9 mA @5 V, white ~0.7 ... 2.6 mA per LED (shared, unballasted) Q1 base: (VCC - Veb) / 3.3k = 0.8 ... 1.3 mA, forced beta ~9-15 at <= 20 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"
- note removed: "Astable 555. Q1 (PNP) turns on while OUT is LOW (discharge phase). t_on = 0.693 * R2 * C1 = 83 ms t_off = 0.693 * (R1 + R2) * C1 = 776 ms f = 1.16 Hz, LED duty 9.7 % I_digit = (VCC - Vce_sat - Vf) / R: E 680R, C 820R -> ~0.4 mA @3.3 V ... ~0.9 mA @5 V average per LED (shared, unballasted) Q1 base: (VCC - Veb) / 4.7k = 0.55 ... 0.9 mA, forced beta >= 10"
Changed lines of the file:
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@@
 		(comment 1 "CMOS 555 astable, 14 orange LEDs sink to OUT (lit when OUT low)")
 	)
-	(text "D1-D14 placed on BOTTOM side spelling \"ECE\" (7-segment layout)."
+	(text "Astable 555. Q1 (PNP) turns on while OUT is LOW (discharge phase).\nt_on  = 0.693 * R2 * C1          = 83 ms\nt_off = 0.693 * (R1 + R2) * C1   = 776 ms\nf = 1.16 Hz, LED duty 9.7 %\nI_digit = (VCC - Vce_sat - Vf) / R:  E (orange) 680R, C (white) 220R\n  orange ~0.4 mA @3.3 V ... ~0.9 mA @5 V, white ~0.7 ... 2.6 mA per LED (shared, unballasted)\nQ1 base: (VCC - Veb) / 3.3k = 0.8 ... 1.3 mA, forced beta ~9-15 at <= 20 mA"
 		(exclude_from_sim no)
-		(at 76.2 167.64 0)
+		(at 30.48 35.56 0)
 		(effects
 			(font
@@
 		)
 	)
-	(text "Astable 555. Q1 (PNP) turns on while OUT is LOW (discharge phase).\nt_on  = 0.693 * R2 * C1          = 83 ms\nt_off = 0.693 * (R1 + R2) * C1   = 776 ms\nf = 1.16 Hz, LED duty 9.7 %\nI_digit = (VCC - Vce_sat - Vf) / R:  E 680R, C 820R\n  -> ~0.4 mA @3.3 V ... ~0.9 mA @5 V average per LED (shared, unballasted)\nQ1 base: (VCC - Veb) / 4.7k = 0.55 ... 0.9 mA, forced beta >= 10"
+	(text "D1-D14 placed on BOTTOM side spelling \"ECE\" (7-segment layout)."
 		(exclude_from_sim no)
-		(at 30.48 35.56 0)
+		(at 76.2 167.64 0)
 		(effects
 			(font
@@
 			)
 		)
-		(property "Value" "Orange"
+		(property "Value" "White"
 			(at 145.42 149.86 90)
 			(hide yes)
@@
 			)
 		)
-		(property "Description" "Orange 605 nm 0603 LED (XINGLIGHT)"
+		(property "Description" "White 0603 LED, Vf 2.7 V @ 20 mA (XINGLIGHT)"
 			(at 149.86 147.32 90)
 			(hide yes)
@@
 			)
 		)
-		(property "LCSC" "C965800"
+		(property "LCSC" "C965808"
 			(at 149.86 147.32 90)
 			(hide yes)
@@
 			)
 		)
-		(property "MPN" "XL-1608UOC-06"
+		(property "MPN" "XL-1608UWC-04"
 			(at 149.86 147.32 90)
 			(hide yes)
@@
 			)
 		)
-		(property "Value" "Orange"
+		(property "Value" "White"
 			(at 158.12 149.86 90)
 			(hide yes)
@@
 			)
 		)
-		(property "Description" "Orange 605 nm 0603 LED (XINGLIGHT)"
+		(property "Description" "White 0603 LED, Vf 2.7 V @ 20 mA (XINGLIGHT)"
 			(at 162.56 147.32 90)
 			(hide yes)
@@
 			)
 		)
-		(property "LCSC" "C965800"
+		(property "LCSC" "C965808"
 			(at 162.56 147.32 90)
 			(hide yes)
@@
 			)
 		)
-		(property "MPN" "XL-1608UOC-06"
+		(property "MPN" "XL-1608UWC-04"
 			(at 162.56 147.32 90)
 			(hide yes)
@@
 			)
 		)
-		(property "Value" "4.7k"
+		(property "Value" "3.3k"
 			(at 64.77 115.57 90)
 			(show_name no)
@@
 			)
 		)
-		(property "Description" "4.7 kOhm 1% 0603, Q1 base (forced beta >= 10 at 3.3-5 V)"
+		(property "Description" "3.3 kOhm 1% 0603, Q1 base (forced beta ~9-15 at 3.3-5 V, ~20 mA load)"
 			(at 66.04 111.76 90)
 			(hide yes)
@@
 			)
 		)
-		(property "LCSC" "C23162"
+		(property "LCSC" "C22978"
 			(at 66.04 111.76 90)
 			(hide yes)
@@
 			)
 		)
-		(property "MPN" "0603WAF4701T5E"
+		(property "MPN" "0603WAF3301T5E"
 			(at 66.04 111.76 90)
 			(hide yes)
@@
 			)
 		)
-		(property "Value" "Orange"
+		(property "Value" "White"
 			(at 183.52 149.86 90)
 			(hide yes)
@@
 			)
 		)
-		(property "Description" "Orange 605 nm 0603 LED (XINGLIGHT)"
+		(property "Description" "White 0603 LED, Vf 2.7 V @ 20 mA (XINGLIGHT)"
 			(at 187.96 147.32 90)
 			(hide yes)
@@
 			)
 		)
-		(property "LCSC" "C965800"
+		(property "LCSC" "C965808"
 			(at 187.96 147.32 90)
 			(hide yes)
@@
 			)
 		)
-		(property "MPN" "XL-1608UOC-06"
+		(property "MPN" "XL-1608UWC-04"
 			(at 187.96 147.32 90)
 			(hide yes)
@@
 			)
 		)
-		(property "Value" "820"
+		(property "Value" "220"
 			(at 172.72 123.19 0)
 			(show_name no)
@@
 			)
 		)
-		(property "Description" "820 Ohm 1% 0603, digit C (4 LEDs)"
+		(property "Description" "220 Ohm 1% 0603, digit C (4 white LEDs)"
 			(at 170.18 121.92 0)
 			(hide yes)
@@
 			)
 		)
-		(property "LCSC" "C23253"
+		(property "LCSC" "C22962"
 			(at 170.18 121.92 0)
 			(hide yes)
@@
 			)
 		)
-		(property "MPN" "0603WAF8200T5E"
+		(property "MPN" "0603WAF2200T5E"
 			(at 170.18 121.92 0)
 			(hide yes)
@@
 			)
 		)
-		(property "Value" "Orange"
+		(property "Value" "White"
 			(at 170.82 149.86 90)
 			(hide yes)
@@
 			)
 		)
-		(property "Description" "Orange 605 nm 0603 LED (XINGLIGHT)"
+		(property "Description" "White 0603 LED, Vf 2.7 V @ 20 mA (XINGLIGHT)"
 			(at 175.26 147.32 90)
 			(hide yes)
@@
 			)
 		)
-		(property "LCSC" "C965800"
+		(property "LCSC" "C965808"
 			(at 175.26 147.32 90)
 			(hide yes)
@@
 			)
 		)
-		(property "MPN" "XL-1608UOC-06"
+		(property "MPN" "XL-1608UWC-04"
 			(at 175.26 147.32 90)
 			(hide yes)
